File: eagle/wiring.sch (EAGLE design)
At the start: 2 parts

Commit message: Clean up for report
Parts:
- removed S1: (no value), switch-omron:31-XX
- added SWITCH: (no value), switch-omron:31-XX
Connections:
- net NEUTRAL renamed AC/N
- removed net LIVE_PANEL: S1.P
- new net AC/L: SWITCH.P
- net LIVE_LIGHT: now also SWITCH.S; no longer S1.S
Other:
- note added: "FAN"
- note added: "TIMER"
- note added: "To panel"
- note removed: "Fan"
- note removed: "Timer"
- moved on the sheet: LIGHT
